File: theresynth.sch (KiCad schematic (older format))
At the start: 87 parts, among them J1 Jack-12V AC, J2 AudioJack2, J3 AudioJack2, Q1 2N3904, Q2 2N3904, Q3 2N3904, Q4 2N3904, Q5 2N3904, Q6 J111, U1 TL074, U2 LM78L12_TO92, U3 LM79L12_TO92

Commit message: completely connected
Parts:
- added C19, C20: 100n, Capacitor_THT:C_Rect_L7.2mm_W2.5mm_P5.00mm_FKS2_FKP2_MKS2_MKP2, symbol Device:C
- added D1: LED, LED_THT:LED_D3.0mm, symbol Device:LED_Dual_2pin
- added D7: LED, LED_THT:LED_D3.0mm, symbol Device:LED
- added J5: External Ground, Connector_Pin:Pin_D1.4mm_L8.5mm_W2.8mm_FlatFork, symbol Connector:Conn_01x01_Female
- added R32, R51: 1k, Resistor_THT:R_Axial_DIN0204_L3.6mm_D1.6mm_P7.62mm_Horizontal, symbol Device:R
- added R34: 5k, Resistor_THT:R_Axial_DIN0204_L3.6mm_D1.6mm_P7.62mm_Horizontal, symbol Device:R
- added R35: 10k, Resistor_THT:R_Axial_DIN0204_L3.6mm_D1.6mm_P7.62mm_Horizontal, symbol Device:R
- added RV4: 100k, Potentiometer_THT:Potentiometer_Bourns_3296W_Vertical, symbol Device:R_POT
- added SW1: SW_SPST, Eurorack:Horizontal_SPDT_2MS5T2B2M7RE, symbol Switch:SW_SPST
- added U2: TL074, Package_DIP:DIP-14_W7.62mm_LongPads, symbol Amplifier_Operational:TL074
- C3: footprint Capacitor_THT:C_Rect_L7.0mm_W6.5mm_P5.00mm -> Eurorack:Variable_Capacitor_W6.5mm_P5.00mm
- RV3: value R_POT -> 100k
- renumbered C19 to C21, C20 to C22, C25 to C23, C21 to C24, C22 to C25, C23 to C26, C24 to C27, C26 to C28, C27 to C29, C28 to C30, D1 to D2, D2 to D3, D3 to D4, J3 to J2, J2 to J3, R30 to R27, R27 to R28, R28 to R29, R29 to R30, R32 to R33, R34 to R36, R33 to R37, U2 to U3, U3 to U4
Connections:
- wire segments 121 -> 139
Other:
- note added: "VC2 out"
- note removed: "VC out"
- moved on the sheet: AE1, C1, C10, C11, C12, C13, C14, C15, C16, C17, C18, C2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

Commit message: add phones output
Parts:
- added J6: AudioJack3_Switch, Connector_Audio:Jack_3.5mm_Ledino_KB3SPRS_Horizontal, symbol Connector:AudioJack3_SwitchTR
- added R52: 1k, Resistor_THT:R_Axial_DIN0204_L3.6mm_D1.6mm_P7.62mm_Horizontal, symbol Device:R
- added RV8: 100k, Potentiometer_THT:Potentiometer_Alps_RK163_Single_Horizontal, symbol Device:R_POT
- added U5: TL074, Package_DIP:DIP-14_W7.62mm_LongPads, symbol Amplifier_Operational:TL074
- C24, C25: value 2200u -> 4700u
- J5: value External Ground -> Ext. GND
- U3: value LM78L12_TO92 -> LM7812_TO220; footprint Package_TO_SOT_THT:TO-92_Inline_Wide -> Package_TO_SOT_THT:TO-220-3_Vertical; symbol Regulator_Linear:LM78L12_TO92 -> Regulator_Linear:LM7812_TO220
- U4: value LM79L12_TO92 -> LM7912_TO220; footprint Package_TO_SOT_THT:TO-92_Inline_Wide -> Package_TO_SOT_THT:TO-220-3_Vertical; symbol Regulator_Linear:LM79L12_TO92 -> Regulator_Linear:LM7912_TO220
Connections:
- wire segments 139 -> 150
Other:
- moved on the sheet: D7, J5, R51
Changed lines of the file:
@@
 P 9150 5750
 F 0 "C24" H 9268 5796 50  0000 L CNN
-F 1 "2200u" H 9268 5705 50  0000 L CNN
+F 1 "4700u" H 9268 5705 50  0000 L CNN
 F 2 "Capacitor_THT:C_Radial_D16.0mm_H31.5mm_P7.50mm" H 9188 5600 50  0001 C CNN
 F 3 "~" H 9150 5750 50  0001 C CNN
@@
 P 9150 6050
 F 0 "C25" H 9268 6096 50  0000 L CNN
-F 1 "2200u" H 9268 6005 50  0000 L CNN
+F 1 "4700u" H 9268 6005 50  0000 L CNN
 F 2 "Capacitor_THT:C_Radial_D16.0mm_H31.5mm_P7.50mm" H 9188 5900 50  0001 C CNN
 F 3 "~" H 9150 6050 50  0001 C CNN
@@
 $EndComp
 $Comp
-L Regulator_Linear:LM79L12_TO92 U4
+L Regulator_Linear:LM7912_TO220 U4
 U 1 1 5F34F527
 P 9900 6200
 F 0 "U4" H 9900 6051 50  0000 C CNN
-F 1 "LM79L12_TO92" H 9900 5960 50  0000 C CNN
-F 2 "Package_TO_SOT_THT:TO-92_Inline_Wide" H 9900 6000 50  0001 C CIN
+F 1 "LM7912_TO220" H 9900 5960 50  0000 C CNN
+F 2 "Package_TO_SOT_THT:TO-220-3_Vertical" H 9900 6000 50  0001 C CIN
 F 3 "http://www.ti.com/lit/ds/symlink/lm79l.pdf" H 9900 6200 50  0001 C CNN
 	1    9900 6200
@@
 Connection ~ 9900 5900
 $Comp
-L Regulator_Linear:LM78L12_TO92 U3
+L Regulator_Linear:LM7812_TO220 U3
 U 1 1 5F3473C8
 P 9900 5600
 F 0 "U3" H 9900 5842 50  0000 C CNN
-F 1 "LM78L12_TO92" H 9900 5751 50  0000 C CNN
-F 2 "Package_TO_SOT_THT:TO-92_Inline_Wide" H 9900 5825 50  0001 C CIN
+F 1 "LM7812_TO220" H 9900 5751 50  0000 C CNN
+F 2 "Package_TO_SOT_THT:TO-220-3_Vertical" H 9900 5825 50  0001 C CIN
 F 3 "http://www.fairchildsemi.com/ds/LM/LM78L05A.pdf" H 9900 5550 50  0001 C CNN
 	1    9900 5600
@@
 	1    0    0    -1
 $EndComp
-Wire Wire Line
-	7450 2150 7650 2150
 Wire Wire Line
 	7650 2350 7650 2500
@@
 	7000 3500 7000 2750
 Wire Wire Line
-	7450 2150 7450 2850
-Wire Wire Line
-	7450 2850 10050 2850
-Wire Wire Line
-	10050 2850 10050 3150
-Connection ~ 10050 3150
-Wire Wire Line
 	10400 2250 10400 2550
 Wire Wire Line
@@
 L Device:R R51
 U 1 1 5FA5917F
-P 10150 5150
-F 0 "R51" V 9943 5150 50  0000 C CNN
-F 1 "1k" V 10034 5150 50  0000 C CNN
-F 2 "Resistor_THT:R_Axial_DIN0204_L3.6mm_D1.6mm_P7.62mm_Horizontal" V 10080 5150 50  0001 C CNN
-F 3 "~" H 10150 5150 50  0001 C CNN
-	1    10150 5150
+P 6000 7650
+F 0 "R51" V 5793 7650 50  0000 C CNN
+F 1 "1k" V 5884 7650 50  0000 C CNN
+F 2 "Resistor_THT:R_Axial_DIN0204_L3.6mm_D1.6mm_P7.62mm_Horizontal" V 5930 7650 50  0001 C CNN
+F 3 "~" H 6000 7650 50  0001 C CNN
+	1    6000 7650
 	0    1    1    0
 $EndComp
@@
 L power:+12V #PWR058
 U 1 1 5FA5B505
-P 10000 5150
-F 0 "#PWR058" H 10000 5000 50  0001 C CNN
-F 1 "+12V" V 10015 5278 50  0000 L CNN
-F 2 "" H 10000 5150 50  0001 C CNN
-F 3 "" H 10000 5150 50  0001 C CNN
-	1    10000 5150
+P 5850 7650
+F 0 "#PWR058" H 5850 7500 50  0001 C CNN
+F 1 "+12V" V 5865 7778 50  0000 L CNN
+F 2 "" H 5850 7650 50  0001 C CNN
+F 3 "" H 5850 7650 50  0001 C CNN
+	1    5850 7650
 	0    -1   -1   0
 $EndComp
@@
 L Device:LED D7
 U 1 1 5FA5C82A
-P 10450 5150
-F 0 "D7" H 10443 4895 50  0000 C CNN
-F 1 "LED" H 10443 4986 50  0000 C CNN
-F 2 "LED_THT:LED_D3.0mm" H 10450 5150 50  0001 C CNN
-F 3 "~" H 10450 5150 50  0001 C CNN
-	1    10450 5150
+P 6300 7650
+F 0 "D7" H 6293 7395 50  0000 C CNN
+F 1 "LED" H 6293 7486 50  0000 C CNN
+F 2 "LED_THT:LED_D3.0mm" H 6300 7650 50  0001 C CNN
+F 3 "~" H 6300 7650 50  0001 C CNN
+	1    6300 7650
 	-1   0    0    1
 $EndComp
@@
 L power:GND #PWR059
 U 1 1 5FA5DFA6
-P 10700 5150
-F 0 "#PWR059" H 10700 4900 50  0001 C CNN
-F 1 "GND" V 10705 5022 50  0000 R CNN
-F 2 "" H 10700 5150 50  0001 C CNN
-F 3 "" H 10700 5150 50  0001 C CNN
-	1    10700 5150
+P 6550 7650
+F 0 "#PWR059" H 6550 7400 50  0001 C CNN
+F 1 "GND" V 6555 7522 50  0000 R CNN
+F 2 "" H 6550 7650 50  0001 C CNN
+F 3 "" H 6550 7650 50  0001 C CNN
+	1    6550 7650
 	0    -1   -1   0
 $EndComp
 Wire Wire Line
-	10700 5150 10600 5150
+	6550 7650 6450 7650
 $Comp
 L Connector:Conn_01x01_Female J5
 U 1 1 5F62A036
-P 10400 4550
-F 0 "J5" H 10428 4576 50  0000 L CNN
-F 1 "External Ground" H 10428 4485 50  0000 L CNN
-F 2 "Connector_Pin:Pin_D1.4mm_L8.5mm_W2.8mm_FlatFork" H 10400 4550 50  0001 C CNN
-F 3 "~" H 10400 4550 50  0001 C CNN
-	1    10400 4550
+P 6450 6700
+F 0 "J5" H 6478 6726 50  0000 L CNN
+F 1 "Ext. GND" H 6478 6635 50  0000 L CNN
+F 2 "Connector_Pin:Pin_D1.4mm_L8.5mm_W2.8mm_FlatFork" H 6450 6700 50  0001 C CNN
+F 3 "~" H 6450 6700 50  0001 C CNN
+	1    6450 6700
 	1    0    0    -1
 $EndComp
@@
 L power:GND #PWR060
 U 1 1 5F62B318
-P 10200 4550
-F 0 "#PWR060" H 10200 4300 50  0001 C CNN
-F 1 "GND" V 10205 4422 50  0000 R CNN
-F 2 "" H 10200 4550 50  0001 C CNN
-F 3 "" H 10200 4550 50  0001 C CNN
-	1    10200 4550
-	0    1    1    0
+P 6250 6700
+F 0 "#PWR060" H 6250 6450 50  0001 C CNN
+F 1 "GND" V 6255 6572 50  0000 R CNN
+F 2 "" H 6250 6700 50  0001 C CNN
+F 3 "" H 6250 6700 50  0001 C CNN
+	1    6250 6700
+	0    1    1    0
+$EndComp
+Wire Wire Line
+	6700 2750 6700 2150
+Wire Wire Line
+	6700 2150 7650 2150
+Wire Wire Line
+	9150 4850 9350 4850
+Wire Wire Line
+	8550 5200 8550 4950
+Wire Wire Line
+	8550 5200 9150 5200
+Wire Wire Line
+	9150 5200 9150 4850
+Connection ~ 9150 4850
+$Comp
+L Amplifier_Operational:TL074 U?
+U 4 1 5F664AB7
+P 8850 4850
+AR Path="/5F35ADD1/5F664AB7" Ref="U?"  Part="4"
+AR Path="/5F664AB7" Ref="U5"  Part="4"
+F 0 "U5" H 8850 5217 50  0000 C CNN
+F 1 "TL074" H 8850 5126 50  0000 C CNN
+F 2 "Package_DIP:DIP-14_W7.62mm_LongPads" H 8800 4950 50  0001 C CNN
+F 3 "http://www.ti.com/lit/ds/symlink/tl071.pdf" H 8900 5050 50  0001 C CNN
+	4    8850 4850
+	1    0    0    -1
+$EndComp
+$Comp
+L Device:R R52
+U 1 1 5F67993B
+P 9500 4850
+F 0 "R52" V 9293 4850 50  0000 C CNN
+F 1 "1k" V 9384 4850 50  0000 C CNN
+F 2 "Resistor_THT:R_Axial_DIN0204_L3.6mm_D1.6mm_P7.62mm_Horizontal" V 9430 4850 50  0001 C CNN
+F 3 "~" H 9500 4850 50  0001 C CNN
+	1    9500 4850
+	0    1    1    0
+$EndComp
+$Comp
+L Connector:AudioJack3_SwitchTR J6
+U 1 1 5F67FA53
+P 10350 4700
+F 0 "J6" H 10070 4533 50  0000 R CNN
+F 1 "AudioJack3_Switch" H 10070 4624 50  0000 R CNN
+F 2 "Connector_Audio:Jack_3.5mm_Ledino_KB3SPRS_Horizontal" H 10350 4700 50  0001 C CNN
+F 3 "~" H 10350 4700 50  0001 C CNN
+	1    10350 4700
+	-1   0    0    1
+$EndComp
+$Comp
+L power:GND #PWR0101
+U 1 1 5F68BE9B
+P 10150 4800
+F 0 "#PWR0101" H 10150 4550 50  0001 C CNN
+F 1 "GND" H 10155 4627 50  0000 C CNN
+F 2 "" H 10150 4800 50  0001 C CNN
+F 3 "" H 10150 4800 50  0001 C CNN
+	1    10150 4800
+	1    0    0    -1
+$EndComp
+Wire Wire Line
+	10150 4700 10050 4700
+Wire Wire Line
+	10150 4500 10050 4500
+Wire Wire Line
+	10050 4500 10050 4700
+Connection ~ 10050 4700
+Wire Wire Line
+	10050 4700 9800 4700
+Wire Wire Line
+	10050 4000 10050 4400
+Wire Wire Line
+	10050 4400 9550 4400
+Wire Wire Line
+	9550 4400 9550 4600
+Wire Wire Line
+	9550 4600 8550 4600
+Wire Wire Line
+	8550 4600 8550 4750
+Connection ~ 10050 4000
+$Comp
+L Device:R_POT RV8
+U 1 1 5F6ECCE5
+P 9800 4850
+F 0 "RV8" V 9593 4850 50  0000 C CNN
+F 1 "100k" V 9684 4850 50  0000 C CNN
+F 2 "Potentiometer_THT:Potentiometer_Alps_RK163_Single_Horizontal" H 9800 4850 50  0001 C CNN
+F 3 "~" H 9800 4850 50  0001 C CNN
+	1    9800 4850
+	-1   0    0    1
+$EndComp
+$Comp
+L power:GND #PWR0102
+U 1 1 5F711D98
+P 9800 5000
+F 0 "#PWR0102" H 9800 4750 50  0001 C CNN
+F 1 "GND" H 9805 4827 50  0000 C CNN
+F 2 "" H 9800 5000 50  0001 C CNN
+F 3 "" H 9800 5000 50  0001 C CNN
+	1    9800 5000
+	1    0    0    -1
 $EndComp
 $EndSCHEMATC

Commit message: removed 2 opamp units
Parts:
- removed C24, C25: 4700u, Capacitor_THT:C_Radial_D16.0mm_H31.5mm_P7.50mm, symbol Device:CP
- removed C27: 1u, Capacitor_THT:C_Rect_L7.0mm_W6.0mm_P5.00mm, symbol Device:C
- removed C29, C30: 100n, Capacitor_THT:C_Rect_L7.2mm_W2.5mm_P5.00mm_FKS2_FKP2_MKS2_MKP2, symbol Device:C
- removed D2, D3: 1N4001, Diode_THT:D_DO-35_SOD27_P7.62mm_Horizontal, symbol Diode:1N4001
- removed D7: LED, LED_THT:LED_D3.0mm, symbol Device:LED
- removed J1: Jack-12V AC, Connector_BarrelJack:BarrelJack_Horizontal, symbol Connector:Jack-DC
- removed J5: Ext. GND, Connector_Pin:Pin_D1.4mm_L8.5mm_W2.8mm_FlatFork, symbol Connector:Conn_01x01_Female
- removed R23: 47k, Resistor_THT:R_Axial_DIN0204_L3.6mm_D1.6mm_P7.62mm_Horizontal, symbol Device:R
- removed R24: 9.52k, Resistor_THT:R_Axial_DIN0204_L3.6mm_D1.6mm_P7.62mm_Horizontal, symbol Device:R
- removed R51: 1k, Resistor_THT:R_Axial_DIN0204_L3.6mm_D1.6mm_P7.62mm_Horizontal, symbol Device:R
- removed SW1: SW_SPST, Eurorack:Horizontal_SPDT_2MS5T2B2M7RE, symbol Switch:SW_SPST
- removed unit 1 of U1
- removed U3: LM7812_TO220, Package_TO_SOT_THT:TO-220-3_Vertical, symbol Regulator_Linear:LM7812_TO220
- removed U4: LM7912_TO220, Package_TO_SOT_THT:TO-220-3_Vertical, symbol Regulator_Linear:LM7912_TO220
- added C18: 10n, Capacitor_THT:C_Rect_L7.2mm_W2.5mm_P5.00mm_FKS2_FKP2_MKS2_MKP2, symbol Device:C
- added J7: To_Amp, Connector_PinHeader_2.54mm:PinHeader_1x03_P2.54mm_Vertical, symbol Connector:Conn_01x03_Male
- added R22: 2.2k, Resistor_THT:R_Axial_DIN0204_L3.6mm_D1.6mm_P7.62mm_Horizontal, symbol Device:R
- added R5: 220, Resistor_THT:R_Axial_DIN0204_L3.6mm_D1.6mm_P7.62mm_Horizontal, symbol Device:R
- added RV10: 100k, Potentiometer_THT:Potentiometer_Alps_RK163_Single_Horizontal, symbol Device:R_POT
- added RV4, RV6: 10k, Potentiometer_THT:Potentiometer_Vishay_T73YP_Vertical, symbol Device:R_POT
- added TP1, TP2, TP3: TestPoint, TestPoint:TestPoint_THTPad_1.0x1.0mm_Drill0.5mm, symbol Connector:TestPoint
- C1: value 33p -> 22p
- C19: renamed from C18; value 100n -> 1u; footprint Capacitor_THT:C_Rect_L7.2mm_W2.5mm_P5.00mm_FKS2_FKP2_MKS2_MKP2 -> Capacitor_THT:C_Rect_L7.0mm_W6.0mm_P5.00mm
- C2: value 47p -> 22p
- C23: renamed from C22; value 40n -> 10n
- C3: value 60p -> 20p
- Q6: value J111 -> J113; symbol Device:Q_NJFET_GDS -> Device:Q_NJFET_DSG
- R23: renamed from R21; value 1k -> 10k
- R26: renamed from R22; value 100k -> 10k
- R27: renamed from R35; value 10k -> 100k
- R31: renamed from R27; value 10k -> 100k
- R36: renamed from R34; value 5k -> 1k
- U3: renamed from U2; value TL074 -> TL072; footprint Package_DIP:DIP-14_W7.62mm_LongPads -> Package_DIP:DIP-8_W7.62mm_LongPads; symbol Amplifier_Operational:TL074 -> Amplifier_Operational:TL072
- renumbered C19 to C20, C20 to C21, C21 to C22, C23 to C24, C26 to C25, C28 to C26, D4 to D2, J6 to J1, R9 to R10, R10 to R11, R11 to R12, R12 to R13, R13 to R14, R14 to R15, R15 to R16, R16 to R17, R17 to R18, R18 to R19, R19 to R20, R20 to R21, R26 to R28, R28 to R29, R29 to R30, R30 to R32, R31 to R33, R32 to R34, R33 to R35, R52 to R37, R36 to R38, R37 to R39, R5 to R6, R6 to R7, R7 to R8, R8 to R9, RV4 to RV5, RV8 to RV7, U2 to U1, U5 to U2
Connections:
- net +12V: now also J7.1 (Pin_1)
- net GND: now also Q6.2 (S), R31.1, C18.2, J7.2 (Pin_2), RV10.1; no longer C23.1, Q6.3 (S)
- net VolumeControlOut: now also RV4.1
- net at R26.2: now also R27.2, U1.2 (-); no longer C19.1
- net at C8.2, C9.1: now also R5.2; no longer RV1.1
- net at C17.2, Q5.3 (C), R20.2: now also R22.1; no longer C19.2
- net at C14.1, Q3.1 (E), R15.1: now also TP1.1
- net at C15.2, Q4.1 (E), R16.1: now also TP2.1
- net at R25.2: now also RV3.1; no longer U1.12 (+)
- net at R23.1, RV3.3: no longer RV3.2
- net at R25.1, U1.5 (+): now also Q6.1 (D); no longer Q6.2 (D)
- net at C22.2: now also Q6.3 (G), RV4.2, RV4.3; no longer Q6.1 (G)
- net at R38.1: now also RV10.2; no longer J2.T
- net at R39.2, U1.14: now also U3.5 (+), RV6.2, RV6.3; no longer R27.1, U3.10 (+)
- net at J1.TN: now also J7.3 (Pin_3)
- net at R36.2, U1.13 (-): now also RV6.1; no longer R27.2
- new net: C19.1, RV3.2, TP3.1, U1.3 (+)
- new net: C18.1, C19.2, R22.2
- new net: R5.1, RV1.1
- new net: J2.T, RV10.3
- new net: C23.2, R27.1, U1.1
- new net: C23.1, D2.2 (A), R31.2
- new net: R34.2, U3.6 (-), U3.7
Other:
- note added: "CV2 out"
- note added: "Overdrive"
- note added: "TODO: potenziometro pin2 ai 2 condensatori?"
- note added: "TODO: remove?"
- note added: "TODO: si puo' togliere ultmo filtro?"
- note removed: "Shape amplifier / Overdrive"
- note removed: "VC2 out"
- moved on the sheet: C13, C23, J1, J2, Q4, R10, R13, R14, R16, R23, R25, R26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

Commit message: full connection before relayouting labels
Parts:
- removed C18: 10n, Capacitor_THT:C_Rect_L7.2mm_W2.5mm_P5.00mm_FKS2_FKP2_MKS2_MKP2, symbol Device:C
- removed C20, C21: 100n, Capacitor_THT:C_Rect_L7.2mm_W2.5mm_P5.00mm_FKS2_FKP2_MKS2_MKP2, symbol Device:C
- removed R19: 1k, Resistor_THT:R_Axial_DIN0204_L3.6mm_D1.6mm_P7.62mm_Horizontal, symbol Device:R
- removed unit 5 of U1
- J7: footprint Connector_PinHeader_2.54mm:PinHeader_1x03_P2.54mm_Vertical -> Connector_PinHeader_2.54mm:PinHeader_1x04_P2.54mm_Vertical; symbol Connector:Conn_01x03_Male -> Connector:Conn_01x04_Male
- R17: value 260k -> 470k
- R18: value 100k -> 47k
- R20: value 6.8k -> 10k
- R22: value 2.2k -> 1M
- R23: value 10k -> 22k
- R5: value 220 -> 1k
- RV1: value 1k -> 100k
Connections:
- net +12V: now also C16.1, C17.1, J7.3 (Pin_3), R17.1, R20.1, RV1.1; no longer J7.1 (Pin_1)
- net -12V: now also J7.4 (Pin_4), RV1.3
- net GND: now also J7.1 (Pin_1); no longer J7.2 (Pin_2)
- net at C13.2, Q2.1 (E), R10.1: now also R5.1; no longer RV1.2, RV1.3
- net at C5.1, C8.1, Q2.2 (B)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: now also R22.1
- net at C17.2, Q5.3 (C), R20.2: now also C19.2; no longer R22.1
- net at R22.2: now also RV1.2; no longer C19.2
- net at C26.1, U1.8, U1.9 (-)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: now also RV10.3; no longer R38.2
- net at R38.1: now also J2.T; no longer RV10.2
- net at U2.13 (-), U2.14: now also RV7.3; no longer R37.2
- net at R37.1: now also J1.R, J1.T; no longer RV7.2
- net at J1.TN: now also J7.2 (Pin_2); no longer J7.3 (Pin_3)
- net VolumeControlOut renamed Volume Control/VolumeControlOut
- new net: R38.2, RV10.2
- new net: R37.2, RV7.2
Other:
- note added: "TODO: potenziometro?"
- note added: "TODO:invece dare una tensione alla base con un potenziometro al +12/-12?"
- note removed: "TODO: potenziometro pin2 ai 2 condensatori?"
- note removed: "TODO: remove?"
- moved on the sheet: C19, J1, J2, R37, R38, R5, R6, RV1, RV10, RV7

Commit message: migrate audio processing to new sheet
Parts:
- removed C19, C22, C24: 1u, Capacitor_THT:C_Rect_L7.0mm_W6.0mm_P5.00mm, symbol Device:C
- removed C23, C25, C26: 10n, Capacitor_THT:C_Rect_L7.2mm_W2.5mm_P5.00mm_FKS2_FKP2_MKS2_MKP2, symbol Device:C
- removed D1: LED, LED_THT:LED_D3.0mm, symbol Device:LED_Dual_2pin
- removed D2: 1N4148, Diode_THT:D_DO-35_SOD27_P7.62mm_Horizontal, symbol Diode:1N4148
- removed J1: AudioJack3_Switch, Connector_Audio:Jack_3.5mm_Ledino_KB3SPRS_Horizontal, symbol Connector:AudioJack3_SwitchTR
- removed J2, J3: AudioJack2, Eurorack:PJ302M, symbol Connector:AudioJack2
- removed J7: To_Amp, Connector_PinHeader_2.54mm:PinHeader_1x04_P2.54mm_Vertical, symbol Connector:Conn_01x04_Male
- removed Q6: J113, Package_TO_SOT_THT:TO-92_Inline_Wide, symbol Device:Q_NJFET_DSG
- removed R23, R25: 22k, Resistor_THT:R_Axial_DIN0204_L3.6mm_D1.6mm_P7.62mm_Horizontal, symbol Device:R
- removed R26, R30: 10k, Resistor_THT:R_Axial_DIN0204_L3.6mm_D1.6mm_P7.62mm_Horizontal, symbol Device:R
- removed R27, R29, R31: 100k, Resistor_THT:R_Axial_DIN0204_L3.6mm_D1.6mm_P7.62mm_Horizontal, symbol Device:R
- removed R28: 220k, Resistor_THT:R_Axial_DIN0204_L3.6mm_D1.6mm_P7.62mm_Horizontal, symbol Device:R
- removed R32, R33, R34, R36, R37, R38, R39: 1k, Resistor_THT:R_Axial_DIN0204_L3.6mm_D1.6mm_P7.62mm_Horizontal, symbol Device:R
- removed R35: 1M, Resistor_THT:R_Axial_DIN0204_L3.6mm_D1.6mm_P7.62mm_Horizontal, symbol Device:R
- removed RV10, RV3, RV7: 100k, Potentiometer_THT:Potentiometer_Alps_RK163_Single_Horizontal, symbol Device:R_POT
- removed RV4, RV6: 10k, Potentiometer_THT:Potentiometer_Vishay_T73YP_Vertical, symbol Device:R_POT
- removed RV5: 100k, Potentiometer_THT:Potentiometer_Bourns_3296W_Vertical, symbol Device:R_POT
- removed TP3: TestPoint, TestPoint:TestPoint_THTPad_1.0x1.0mm_Drill0.5mm, symbol Connector:TestPoint
- removed U1, U2: TL074, Package_DIP:DIP-14_W7.62mm_LongPads, symbol Amplifier_Operational:TL074
- removed U3: TL072, Package_DIP:DIP-8_W7.62mm_LongPads, symbol Amplifier_Operational:TL072
- R22: value 1M -> 330k
Connections:
- net Audio Processing/RawAudioIn: now reaches C17.2, Q5.3 (C), R20.2
Other:
- note removed: "Audio filter"
- note removed: "Audio out"
- note removed: "CV2 out"
- note removed: "Overdrive"
- note removed: "TODO: potenziometro?"
- note removed: "TODO: si puo' togliere ultmo filtro?"
- note removed: "TODO:invece dare una tensione alla base con un potenziometro al +12/-12?"
- note removed: "VCA"
- note removed: "Voltage Control from Pitch"
- moved on the sheet: C1, C11, C13, C14, C15, C16, C17, C3, C5, C7, C8, C9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
